Commit message: remove cv_bridge artifacts , add skid steering

File: src/my_robot/urdf/my_robot.xacro (robot description, xacro)
@@ -1,32 +1,44 @@
-<?xml version='1.0'?>
-<robot name="my_robot" xmlns:xacro="http://www.ros.org/wiki/xacro">
+<?xml version="1.0" ?>
+<robot name="Robo4" xmlns:xacro="http://www.ros.org/wiki/xacro">
   <xacro:include filename="$(find my_robot)/urdf/my_robot.gazebo" />
-  <link name="robot_footprint"></link>
-  <joint name="robot_footprint_joint" type="fixed">
-    <origin xyz="0 0 0" rpy="0 0 0" />
-    <parent link="robot_footprint"/>
-    <child link="chassis" />
-  </joint>
-  <link name='chassis'>
-    <pose>0 0 0.1 0 0 0</pose>
-    <inertial>
-      <mass value="15.0"/>
-      <origin xyz="0.0 0 0" rpy=" 0 0 0"/>
-      <inertia
-          ixx="0.1" ixy="0" ixz="0"
-          iyy="0.1" iyz="0"
-          izz="0.1"
-      />
-    </inertial>
-    <collision name='collision'>
-      <origin xyz="0 0 0" rpy=" 0 0 0"/>
-      <geometry>
-        <box size=".4 .2 .1"/>
-      </geometry>
-    </collision>
-    <visual name='chassis_visual'>
-      <origin xyz="0 0 0" rpy=" 0 0 0"/>
-      <geometry>
-        <box size=".4 .2 .1"/>
+  <link name="robot_footprint"/>
+<joint name="robot_footprint_chassis" type="fixed">
+  <origin xyz="0 0 0" rpy="0 0 0" />
+  <parent link="robot_footprint"/>
+  <child link="chassis"/>
+</joint>
+  <link name="chassis">
+    <pose>0 0 0.2 0 0 0</pose>
+    <inertial>
+      <mass value="15"/>
+      <origin rpy="0 0 0" xyz="0 0 0"/>
+      <inertia
+       ixx="0.1" ixy="0" ixz="0"
+       iyy="0.1" iyz="0"
+       izz="0.1"/>
+    </inertial>
+    <collision name="collision">
+      <origin rpy="0 0 0" xyz="0 0 0"/>
+      <geometry>
+        <box size="0.50 0.25 0.1"/>
+      </geometry>
+    </collision>
+    <visual>
+      <origin rpy="0 0 0" xyz="0 0 0"/>
+      <geometry>
+        <box size="0.50 0.25 0.1"/>
+      </geometry>
+    </visual>
+<!--
+    <collision name='front_caster_collision'>
+      <origin xyz="0.15 0 -0.05" rpy=" 0 0 0"/>
+      <geometry>
+        <sphere radius="0.0499"/>
+      </geometry>
+    </collision>
+    <visual name='front_caster_visual'>
+      <origin xyz="0.15 0 -0.05" rpy=" 0 0 0"/>
+      <geometry>
+        <sphere radius="0.05"/>
       </geometry>
     </visual>
@@ -43,92 +55,144 @@
       </geometry>
     </visual>
-    <collision name='front_caster_collision'>
-      <origin xyz="0.15 0 -0.05" rpy=" 0 0 0"/>
-      <geometry>
-        <sphere radius="0.0499"/>
-      </geometry>
-    </collision>
-    <visual name='front_caster_visual'>
-      <origin xyz="0.15 0 -0.05" rpy=" 0 0 0"/>
-      <geometry>
-        <sphere radius="0.05"/>
-      </geometry>
-    </visual>
+-->
   </link>
   <gazebo reference="chassis">
-      <material>Gazebo/Blue</material>
-  </gazebo>
-  <joint type="continuous" name="left_wheel_hinge">
-    <origin xyz="0 0.15 0" rpy="0 0 0"/>
+      <material>Gazebo/Orange</material>
+  </gazebo>
+  <joint name="left_front" type="continuous">
+    <parent link="chassis"/>
     <child link="left_wheel"/>
-    <parent link="chassis"/>
-    <axis xyz="0 1 0" rpy="0 0 0"/>
-    <limit effort="10000" velocity="1000"/>
-    <dynamics damping="1.0" friction="1.0"/>
-  </joint>
-  <link name='left_wheel'>
-    <pose>0 0 0 0 0 0</pose>
-    <inertial>
-      <mass value="5.0"/>
-      <origin xyz="0.0 0 0" rpy=" 0 1.5707 1.5707"/>
-      <inertia
-          ixx="0.1" ixy="0" ixz="0"
-          iyy="0.1" iyz="0"
-          izz="0.1"
-      />
-    </inertial>
-    <collision name='left_wheel_collision'>
-      <origin xyz="0.0 0 0" rpy=" 0 1.5707 1.5707"/>
-      <geometry>
-        <cylinder radius="0.1" length="0.05"/>
-      </geometry>
-    </collision>
-    <visual name='left_wheel_visual'>
-      <origin xyz="0.0 0 0" rpy=" 0 1.5707 1.5707"/>
-      <geometry>
-        <cylinder radius="0.1" length="0.05"/>
+    <origin xyz="0.15 0.15 0.0" rpy="0 0 0"/>
+    <axis xyz="0 1 0"/>
+    <limit effort="10000" velocity="1000"/>
+    <dynamics damping="1.0" friction="1.0"/>
+  </joint>
+  <joint name="right_front" type="continuous">
+    <parent link="chassis"/>
+    <child link="right_wheel"/>
+    <origin xyz="0.15 -0.15 0.0" rpy="0 0 0"/>
+    <axis xyz="0 1 0"/>
+    <limit effort="10000" velocity="1000"/>
+    <dynamics damping="1.0" friction="1.0"/>
+  </joint>
+<!---->
+  <joint name="left_rear" type="continuous">
+    <parent link="chassis"/>
+    <child link="left_rear"/>
+    <origin xyz="-0.15 0.15 0.0" rpy="0 0 0"/>
+    <axis xyz="0 1 0"/>
+    <limit effort="10000" velocity="1000"/>
+    <dynamics damping="1.0" friction="1.0"/>
+  </joint>
+  <joint name="right_rear" type="continuous">
+    <parent link="chassis"/>
+    <child link="right_rear"/>
+    <origin xyz="-0.15 -0.15 0.0" rpy="0 0 0"/>
+    <axis xyz="0 1 0"/>
+    <limit effort="10000" velocity="1000"/>
+    <dynamics damping="1.0" friction="1.0"/>
+  </joint>
+  <link name="left_wheel">
+    <inertial>
+      <mass value="1"/>
+      <origin xyz="0.0 0 0" rpy=" 0 1.5707 1.5707"/>
+      <inertia
+       ixx="0.1" ixy="0" ixz="0"
+       iyy="0.1" iyz="0"
+       izz="0.1"/>
+    </inertial>
+    <collision name="collision">
+      <origin xyz="0.0 0 0" rpy=" 0 1.5707 1.5707"/>
+      <geometry>
+        <cylinder length="0.05" radius="0.1"/>
+      </geometry>
+    </collision>
+    <visual>
+      <origin xyz="0.0 0 0" rpy=" 0 1.5707 1.5707"/>
+      <geometry>
+        <cylinder length="0.05" radius="0.1"/>
       </geometry>
     </visual>
   </link>
   <gazebo reference="left_wheel">
-      <material>Gazebo/Green</material>
-  </gazebo>
-  <joint type="continuous" name="right_wheel_hinge">
-    <origin xyz="0 -0.15 0" rpy="0 0 0"/>
-    <child link="right_wheel"/>
-    <parent link="chassis"/>
-    <axis xyz="0 1 0" rpy="0 0 0"/>
-    <limit effort="10000" velocity="1000"/>
-    <dynamics damping="1.0" friction="1.0"/>
-  </joint>
-  <link name='right_wheel'>
-    <pose>0 0 0 0 0 0</pose>
-    <inertial>
-      <mass value="5.0"/>
-      <origin xyz="0.0 0 0" rpy=" 0 1.5707 1.5707"/>
-      <inertia
-          ixx="0.1" ixy="0" ixz="0"
-          iyy="0.1" iyz="0"
-          izz="0.1"
-      />
-    </inertial>
-    <collision name='right_wheel_collision'>
-      <origin xyz="0.0 0 0" rpy=" 0 1.5707 1.5707"/>
-      <geometry>
-        <cylinder radius="0.1" length="0.05"/>
-      </geometry>
-    </collision>
-    <visual name='right_wheel_visual'>
-      <origin xyz="0.0 0 0" rpy=" 0 1.5707 1.5707"/>
-      <geometry>
-        <cylinder radius="0.1" length="0.05"/>
+      <material>Gazebo/Black</material>
+  </gazebo>
+  <link name="right_wheel">
+    <inertial>
+      <mass value="1"/>
+      <origin xyz="0.0 0 0" rpy=" 0 1.5707 1.5707"/>
+      <inertia
+       ixx="0.1" ixy="0" ixz="0"
+       iyy="0.1" iyz="0"
+       izz="0.1"/>
+    </inertial>
+    <collision name="collision">
+      <origin xyz="0.0 0 0" rpy=" 0 1.5707 1.5707"/>
+      <geometry>
+        <cylinder length="0.05" radius="0.1"/>
+      </geometry>
+    </collision>
+    <visual>
+      <origin xyz="0.0 0 0" rpy=" 0 1.5707 1.5707"/>
+      <geometry>
+        <cylinder length="0.05" radius="0.1"/>
       </geometry>
     </visual>
   </link>
   <gazebo reference="right_wheel">
-      <material>Gazebo/Green</material>
+      <material>Gazebo/Black</material>
+  </gazebo>
+<!---->
+  <link name="left_rear">
+    <inertial>
+      <mass value="1"/>
+      <origin xyz="0.0 0 0" rpy=" 0 1.5707 1.5707"/>
+      <inertia
+       ixx="0.1" ixy="0" ixz="0"
+       iyy="0.1" iyz="0"
+       izz="0.1"/>
+    </inertial>
+    <collision name="collision">
+      <origin xyz="0.0 0 0" rpy=" 0 1.5707 1.5707"/>
+      <geometry>
+        <cylinder length="0.05" radius="0.1"/>
+      </geometry>
+    </collision>
+    <visual>
+      <origin xyz="0.0 0 0" rpy=" 0 1.5707 1.5707"/>
+      <geometry>
+        <cylinder length="0.05" radius="0.1"/>
+      </geometry>
+    </visual>
+  </link>
+  <gazebo reference="left_rear">
+      <material>Gazebo/Black</material>
+  </gazebo>
+  <link name="right_rear">
+    <inertial>
+      <mass value="1"/>
+      <origin xyz="0.0 0 0" rpy=" 0 1.5707 1.5707"/>
+      <inertia
+       ixx="0.1" ixy="0" ixz="0"
+       iyy="0.1" iyz="0"
+       izz="0.1"/>
+    </inertial>
+    <collision name="collision">
+      <origin xyz="0.0 0 0" rpy=" 0 1.5707 1.5707"/>
+      <geometry>
+        <cylinder length="0.05" radius="0.1"/>
+      </geometry>
+    </collision>
+    <visual>
+      <origin xyz="0.0 0 0" rpy=" 0 1.5707 1.5707"/>
+      <geometry>
+        <cylinder length="0.05" radius="0.1"/>
+      </geometry>
+    </visual>
+  </link>
+  <gazebo reference="right_rear">
+      <material>Gazebo/Black</material>
   </gazebo>
   <link name="camera">
-    <pose>0 0 0 0 0 0</pose>
     <inertial>
       <origin xyz="0.0 0.0 0.0" rpy="0.0 0.0 0.0"/>
@@ -139,5 +203,5 @@
       <origin xyz="0.0 0.0 0.0" rpy="0.0 0.0 0.0"/>
       <geometry>
-        <box size="0.05 0.05 0.05"/>
+        <box size="0.05 0.05 0.04"/>
       </geometry>
     </visual>
@@ -145,19 +209,21 @@
       <origin xyz="0.0 0.0 0.0" rpy="0.0 0.0 0.0"/>
       <geometry>
-        <box size="0.05 0.05 0.05"/>
-      </geometry>
-    </collision>
-  </link>
-  <gazebo reference="camera">
-      <material>Gazebo/Red</material>
-  </gazebo>
+        <box size="0.05 0.05 0.04"/>
+      </geometry>
+    </collision>
+  </link>
   <joint name="camera_joint" type="fixed">
-    <origin xyz="0.2 0.0 0.0" rpy="0.0 0.0 0.0"/>
+    <origin xyz="0.25 0.0 0.0" rpy="0.0 0.0 0.0"/>
     <child link="camera"/>
-    <parent link="robot_footprint"/>
+    <parent link="chassis"/>
     <axis xyz="0 1 0" rpy="0 0 0"/>
   </joint>
+  <joint name="hokuyo_joint" type="fixed">
+    <origin xyz="0.225 0.0 0.08" rpy="0.0 0.0 0.0"/>
+    <parent link="chassis"/>
+    <child link="hokuyo"/>
+    <axis xyz="0 1 0"/>
+  </joint>
   <link name="hokuyo">
-    <pose>0 0 0 0 0 0</pose>
     <inertial>
       <origin xyz="0.0 0.0 0.0" rpy="0.0 0.0 0.0"/>
@@ -182,9 +248,6 @@
     </collision>
   </link>
-  <joint name="hokuyo_joint" type="fixed">
-    <origin xyz="0.15 0.0 0.1" rpy="0.0 0.0 0.0"/>
-    <parent link="chassis"/>
-    <child link="hokuyo"/>
-    <axis xyz="0 1 0"/>
-  </joint>
+  <gazebo reference="camera">
+      <material>Gazebo/Blue</material>
+  </gazebo>
 </robot>

Commit message: code complete

File: src/my_robot/urdf/my_robot.xacro (robot description, xacro)
@@ -213,4 +213,12 @@
     </collision>
   </link>
+    <joint name="camera_optical_joint" type="fixed">
+    <origin xyz="0 0 0" rpy="-1.5707 0 -1.5707"/>
+    <parent link="camera"/>
+    <child link="camera_link_optical"/>
+  </joint>
+  <link name="camera_link_optical">
+  </link>
+<!---->
   <joint name="camera_joint" type="fixed">
     <origin xyz="0.25 0.0 0.0" rpy="0.0 0.0 0.0"/>

Commit message: add octomaps, finished localisation, tweak parameters

File: src/my_robot/urdf/my_robot.xacro (robot description, xacro)
@@ -1,4 +1,13 @@
 <?xml version="1.0" ?>
 <robot name="Robo4" xmlns:xacro="http://www.ros.org/wiki/xacro">
+  <material name="blue">
+    <color rgba="0 0 0.8 1"/>
+  </material>
+  <material name="black">
+    <color rgba="0 0 0 1"/>
+  </material>
+  <material name="orange">
+    <color rgba="1 0.5 0.3 1"/>
+  </material>
   <xacro:include filename="$(find my_robot)/urdf/my_robot.gazebo" />
   <link name="robot_footprint"/>
@@ -29,35 +38,68 @@
         <box size="0.50 0.25 0.1"/>
       </geometry>
-    </visual>
-<!--
-    <collision name='front_caster_collision'>
-      <origin xyz="0.15 0 -0.05" rpy=" 0 0 0"/>
-      <geometry>
-        <sphere radius="0.0499"/>
-      </geometry>
-    </collision>
-    <visual name='front_caster_visual'>
-      <origin xyz="0.15 0 -0.05" rpy=" 0 0 0"/>
-      <geometry>
-        <sphere radius="0.05"/>
-      </geometry>
-    </visual>
-    <collision name='back_caster_collision'>
-      <origin xyz="-0.15 0 -0.05" rpy=" 0 0 0"/>
-      <geometry>
-        <sphere radius="0.0499"/>
-      </geometry>
-    </collision>
-    <visual name='back_caster_visual'>
-      <origin xyz="-0.15 0 -0.05" rpy=" 0 0 0"/>
-      <geometry>
-        <sphere radius="0.05"/>
-      </geometry>
-    </visual>
--->
+      <material name="orange"/>
+    </visual>
   </link>
   <gazebo reference="chassis">
       <material>Gazebo/Orange</material>
   </gazebo>
+<joint name="chassis_front_caster" type="fixed">
+  <origin xyz="0 0 0" rpy="0 0 0" />
+  <parent link="chassis"/>
+  <child link="front_caster"/>
+</joint>
+<link name="front_caster">
+    <inertial>
+      <mass value="2"/>
+      <origin xyz="0.20 0 -0.05" rpy=" 0 0 0"/>
+      <inertia
+       ixx="0.01" ixy="0" ixz="0"
+       iyy="0.01" iyz="0"
+       izz="0.01"/>
+    </inertial>
+    <collision name='front_caster_collision'>
+      <origin xyz="0.20 0 -0.05" rpy=" 0 0 0"/>
+      <geometry>
+        <sphere radius="0.0499"/>
+      </geometry>
+    </collision>
+    <visual name='front_caster_visual'>
+      <origin xyz="0.20 0 -0.05" rpy=" 0 0 0"/>
+      <geometry>
+        <sphere radius="0.05"/>
+      </geometry>
+      <material name="black"/>
+    </visual>
+</link>
+<joint name="chassis_back_caster" type="fixed">
+  <origin xyz="0 0 0" rpy="0 0 0" />
+  <parent link="chassis"/>
+  <child link="back_caster"/>
+</joint>
+<link name="back_caster">
+    <inertial>
+      <mass value="2"/>
+      <origin xyz="-0.20 0 -0.05" rpy=" 0 0 0"/>
+      <inertia
+       ixx="0.01" ixy="0" ixz="0"
+       iyy="0.01" iyz="0"
+       izz="0.01"/>
+    </inertial>
+    <collision name='back_caster_collision'>
+      <origin xyz="-0.20 0 -0.05" rpy=" 0 0 0"/>
+      <geometry>
+        <sphere radius="0.0499"/>
+      </geometry>
+    </collision>
+    <visual name='back_caster_visual'>
+      <origin xyz="-0.20 0 -0.05" rpy=" 0 0 0"/>
+      <geometry>
+        <sphere radius="0.05"/>
+      </geometry>
+      <material name="black"/>
+    </visual>
+</link>
+  <xacro:property name="wheel_damping" value="0.5" />
+  <xacro:property name="wheel_friction" value="0.5" />
   <joint name="left_front" type="continuous">
     <parent link="chassis"/>
@@ -66,5 +108,5 @@
     <axis xyz="0 1 0"/>
     <limit effort="10000" velocity="1000"/>
-    <dynamics damping="1.0" friction="1.0"/>
+    <dynamics damping="${wheel_damping}" friction="${wheel_friction}"/>
   </joint>
   <joint name="right_front" type="continuous">
@@ -74,5 +116,5 @@
     <axis xyz="0 1 0"/>
     <limit effort="10000" velocity="1000"/>
-    <dynamics damping="1.0" friction="1.0"/>
+    <dynamics damping="${wheel_damping}" friction="${wheel_friction}"/>
   </joint>
 <!---->
@@ -83,5 +125,5 @@
     <axis xyz="0 1 0"/>
     <limit effort="10000" velocity="1000"/>
-    <dynamics damping="1.0" friction="1.0"/>
+    <dynamics damping="${wheel_damping}" friction="${wheel_friction}"/>
   </joint>
   <joint name="right_rear" type="continuous">
@@ -91,26 +133,35 @@
     <axis xyz="0 1 0"/>
     <limit effort="10000" velocity="1000"/>
-    <dynamics damping="1.0" friction="1.0"/>
-  </joint>
+    <dynamics damping="${wheel_damping}" friction="${wheel_friction}"/>
+  </joint>
+  <xacro:property name="wheel_radius"   value="0.10" />
+  <xacro:property name="wheel_width"    value="0.05" />
+  <xacro:property name="wheel_mass"     value="5" />
+  <xacro:property name="wheel_inertia"  value="${(1/2) * wheel_mass * wheel_radius * wheel_radius }" />
+  <!-- "${(1 / 12) * wheel_mass * ( (3 * wheel_radius * wheel_radius) + (wheel_width * wheel_width ) ) }" -->
+  <xacro:property name="wheel_ixx"   value="0.03" />
+  <xacro:property name="wheel_iyy"   value="${wheel_inertia}" />
+  <xacro:property name="wheel_izz"   value="0.03" />
   <link name="left_wheel">
     <inertial>
-      <mass value="1"/>
-      <origin xyz="0.0 0 0" rpy=" 0 1.5707 1.5707"/>
-      <inertia
-       ixx="0.1" ixy="0" ixz="0"
-       iyy="0.1" iyz="0"
-       izz="0.1"/>
-    </inertial>
-    <collision name="collision">
-      <origin xyz="0.0 0 0" rpy=" 0 1.5707 1.5707"/>
-      <geometry>
-        <cylinder length="0.05" radius="0.1"/>
-      </geometry>
-    </collision>
-    <visual>
-      <origin xyz="0.0 0 0" rpy=" 0 1.5707 1.5707"/>
-      <geometry>
-        <cylinder length="0.05" radius="0.1"/>
-      </geometry>
+      <mass value="${wheel_mass}"/>
+      <origin xyz="0.0 0 0" rpy=" 0 1.5707 1.5707"/>
+      <inertia
+       ixx="${wheel_ixx}" ixy="0" ixz="0"
+       iyy="${wheel_iyy}" iyz="0"
+       izz="${wheel_izz}"/>
+    </inertial>
+    <collision name="collision">
+      <origin xyz="0.0 0 0" rpy=" 0 1.5707 1.5707"/>
+      <geometry>
+        <cylinder length="${wheel_width}" radius="${wheel_radius}"/>
+      </geometry>
+    </collision>
+    <visual>
+      <origin xyz="0.0 0 0" rpy=" 0 1.5707 1.5707"/>
+      <geometry>
+        <cylinder length="${wheel_width}" radius="${wheel_radius}"/>
+      </geometry>
+      <material name="black"/>
     </visual>
   </link>
@@ -120,22 +171,23 @@
   <link name="right_wheel">
     <inertial>
-      <mass value="1"/>
-      <origin xyz="0.0 0 0" rpy=" 0 1.5707 1.5707"/>
-      <inertia
-       ixx="0.1" ixy="0" ixz="0"
-       iyy="0.1" iyz="0"
-       izz="0.1"/>
-    </inertial>
-    <collision name="collision">
-      <origin xyz="0.0 0 0" rpy=" 0 1.5707 1.5707"/>
-      <geometry>
-        <cylinder length="0.05" radius="0.1"/>
-      </geometry>
-    </collision>
-    <visual>
-      <origin xyz="0.0 0 0" rpy=" 0 1.5707 1.5707"/>
-      <geometry>
-        <cylinder length="0.05" radius="0.1"/>
-      </geometry>
+      <mass value="${wheel_mass}"/>
+      <origin xyz="0.0 0 0" rpy=" 0 1.5707 1.5707"/>
+      <inertia
+       ixx="${wheel_ixx}" ixy="0" ixz="0"
+       iyy="${wheel_iyy}" iyz="0"
+       izz="${wheel_izz}"/>
+    </inertial>
+    <collision name="collision">
+      <origin xyz="0.0 0 0" rpy=" 0 1.5707 1.5707"/>
+      <geometry>
+        <cylinder length="${wheel_width}" radius="${wheel_radius}"/>
+      </geometry>
+    </collision>
+    <visual>
+      <origin xyz="0.0 0 0" rpy=" 0 1.5707 1.5707"/>
+      <geometry>
+        <cylinder length="${wheel_width}" radius="${wheel_radius}"/>
+      </geometry>
+      <material name="black"/>
     </visual>
   </link>
@@ -146,22 +198,23 @@
   <link name="left_rear">
     <inertial>
-      <mass value="1"/>
-      <origin xyz="0.0 0 0" rpy=" 0 1.5707 1.5707"/>
-      <inertia
-       ixx="0.1" ixy="0" ixz="0"
-       iyy="0.1" iyz="0"
-       izz="0.1"/>
-    </inertial>
-    <collision name="collision">
-      <origin xyz="0.0 0 0" rpy=" 0 1.5707 1.5707"/>
-      <geometry>
-        <cylinder length="0.05" radius="0.1"/>
-      </geometry>
-    </collision>
-    <visual>
-      <origin xyz="0.0 0 0" rpy=" 0 1.5707 1.5707"/>
-      <geometry>
-        <cylinder length="0.05" radius="0.1"/>
-      </geometry>
+      <mass value="${wheel_mass}"/>
+      <origin xyz="0.0 0 0" rpy=" 0 1.5707 1.5707"/>
+      <inertia
+       ixx="${wheel_ixx}" ixy="0" ixz="0"
+       iyy="${wheel_iyy}" iyz="0"
+       izz="${wheel_izz}"/>
+    </inertial>
+    <collision name="collision">
+      <origin xyz="0.0 0 0" rpy=" 0 1.5707 1.5707"/>
+      <geometry>
+        <cylinder length="${wheel_width}" radius="${wheel_radius}"/>
+      </geometry>
+    </collision>
+    <visual>
+      <origin xyz="0.0 0 0" rpy=" 0 1.5707 1.5707"/>
+      <geometry>
+        <cylinder length="${wheel_width}" radius="${wheel_radius}"/>
+      </geometry>
+      <material name="black"/>
     </visual>
   </link>
@@ -171,22 +224,23 @@
   <link name="right_rear">
     <inertial>
-      <mass value="1"/>
-      <origin xyz="0.0 0 0" rpy=" 0 1.5707 1.5707"/>
-      <inertia
-       ixx="0.1" ixy="0" ixz="0"
-       iyy="0.1" iyz="0"
-       izz="0.1"/>
-    </inertial>
-    <collision name="collision">
-      <origin xyz="0.0 0 0" rpy=" 0 1.5707 1.5707"/>
-      <geometry>
-        <cylinder length="0.05" radius="0.1"/>
-      </geometry>
-    </collision>
-    <visual>
-      <origin xyz="0.0 0 0" rpy=" 0 1.5707 1.5707"/>
-      <geometry>
-        <cylinder length="0.05" radius="0.1"/>
-      </geometry>
+      <mass value="${wheel_mass}"/>
+      <origin xyz="0.0 0 0" rpy=" 0 1.5707 1.5707"/>
+      <inertia
+       ixx="${wheel_ixx}" ixy="0" ixz="0"
+       iyy="${wheel_iyy}" iyz="0"
+       izz="${wheel_izz}"/>
+    </inertial>
+    <collision name="collision">
+      <origin xyz="0.0 0 0" rpy=" 0 1.5707 1.5707"/>
+      <geometry>
+        <cylinder length="${wheel_width}" radius="${wheel_radius}"/>
+      </geometry>
+    </collision>
+    <visual>
+      <origin xyz="0.0 0 0" rpy=" 0 1.5707 1.5707"/>
+      <geometry>
+        <cylinder length="${wheel_width}" radius="${wheel_radius}"/>
+      </geometry>
+      <material name="black"/>
     </visual>
   </link>
@@ -205,4 +259,5 @@
         <box size="0.05 0.05 0.04"/>
       </geometry>
+      <material name="blue"/>
     </visual>
     <collision name="camera_collision">
@@ -259,3 +314,34 @@
       <material>Gazebo/Blue</material>
   </gazebo>
+<!--
+  <joint name="bumper_joint" type="fixed">
+    <origin xyz="0.265 0.0 0.0" rpy="0.0 0.0 0.0"/>
+    <child link="bumper"/>
+    <parent link="chassis"/>
+    <axis xyz="0 1 0" rpy="0 0 0"/>
+  </joint>
+  <link name="bumper">
+    <inertial>
+      <origin xyz="0.0 0.0 0.0" rpy="0.0 0.0 0.0"/>
+      <mass value="0.1"/>
+      <inertia ixx="1e-6" ixy="0" ixz="0" iyy="1e-6" iyz="0" izz="1e-6"/>
+    </inertial>
+    <visual name="bumper_visual">
+      <origin xyz="0.0 0.0 0.0" rpy="0.0 0.0 0.0"/>
+      <geometry>
+        <box size="0.02 0.35 0.1"/>
+      </geometry>
+      <material name="orange"/>
+    </visual>
+    <collision name="bumper_collision">
+      <origin xyz="0.0 0.0 0.0" rpy="0.0 0.0 0.0"/>
+      <geometry>
+        <box size="0.02 0.35 0.1"/>
+      </geometry>
+    </collision>
+  </link>
+  <gazebo reference="bumper">
+      <material>Gazebo/Orange</material>
+  </gazebo>
+-->
 </robot>
